Commit message: Refactor cat URDF and simulation launch for new model
Renamed and refactored the cat URDF Xacro files: 'doraemon.urdf.xacro' is now 'oldcat.xacro', and 'cat.urdf.xacro' is updated to the previous doraemon model. Updated simulation.launch.py to spawn both the mouse and the new cat model, with separate robot descriptions and spawn nodes. This change enables simulation of both the mouse and the updated cat robot in the same environment, and clarifies model naming and topic conventions.

File: oldcat.xacro (robot description, xacro)
@@ -1,4 +1,4 @@
 <?xml version="1.0"?>
-<robot name="doraemon_cat" xmlns:xacro="http://www.ros.org/wiki/xacro">
+<robot name="felix_cat" xmlns:xacro="http://www.ros.org/wiki/xacro">
     <xacro:property name="torso_len" value="0.4"/>
     <xacro:property name="torso_width" value="0.2"/>
@@ -10,9 +10,8 @@
     <xacro:property name="wheel_mass" value="1.0"/>
     <xacro:property name="caster_radius" value="0.04"/>
-    <material name="dora_blue"><color rgba="0.0 0.6 0.9 1"/></material>
-    <material name="dora_white"><color rgba="1 1 1 1"/></material>
-    <material name="dora_red"><color rgba="0.9 0.1 0.1 1"/></material>
-    <material name="dora_yellow"><color rgba="1 0.8 0.1 1"/></material>
+    <material name="blue"> <color rgba="0.16 0.33 0.48 1"/></material>
+    <material name="white"><color rgba="1 1 1 1"/></material>
     <material name="black"><color rgba="0 0 0 1"/></material>
+    <material name="red"><color rgba="0.6941 0.2471 0.3294 1"/></material>
     <material name="silver"><color rgba="0.75 0.75 0.75 1"/></material>
     <xacro:macro name="box_inertia" params="m x y z">
@@ -43,5 +42,5 @@
         <visual>
             <geometry><box size="${torso_len} ${torso_width} ${torso_height}"/></geometry>
-            <material name="dora_blue"/>
+            <material name="blue"/>
         </visual>
         <collision>
@@ -50,21 +49,9 @@
         <xacro:box_inertia m="${torso_mass}" x="${torso_len}" y="${torso_width}" z="${torso_height}"/>
     </link>
-    <gazebo reference="base_link"><material>Gazebo/SkyBlue</material></gazebo>
-    <link name="pocket">
-        <visual>
-            <geometry><box size="0.01 0.14 0.10"/></geometry>
-            <material name="dora_white"/>
-        </visual>
-    </link>
-    <joint name="pocket_joint" type="fixed">
-        <parent link="base_link"/>
-        <child link="pocket"/>
-        <origin xyz="${torso_len/2 + 0.001} 0 0" rpy="0 0 0"/>
-    </joint>
-    <gazebo reference="pocket"><material>Gazebo/White</material></gazebo>
+    <gazebo reference="base_link"><material>Gazebo/Blue</material></gazebo>
     <link name="head">
         <visual>
             <geometry><box size="${head_size} ${head_size} ${head_size}"/></geometry>
-            <material name="dora_blue"/>
+            <material name="blue"/>
         </visual>
         <collision>
@@ -73,5 +60,5 @@
         <xacro:box_inertia m="1.0" x="${head_size}" y="${head_size}" z="${head_size}"/>
     </link>
-    <gazebo reference="head"><material>Gazebo/SkyBlue</material></gazebo>
+    <gazebo reference="head"><material>Gazebo/Blue</material></gazebo>
     <joint name="neck_joint" type="fixed">
         <parent link="base_link"/>
@@ -79,32 +66,8 @@
         <origin xyz="${torso_len/2 + head_size/2 - 0.05} 0 ${torso_height/2 - head_size/4}" rpy="0 0 0"/>
     </joint>
-    <link name="face_mask">
-        <visual>
-            <geometry><box size="0.01 0.13 0.11"/></geometry>
-            <material name="dora_white"/>
-        </visual>
-    </link>
-    <joint name="face_mask_joint" type="fixed">
-        <parent link="head"/>
-        <child link="face_mask"/>
-        <origin xyz="${head_size/2 + 0.001} 0 -0.01" rpy="0 0 0"/>
-    </joint>
-    <gazebo reference="face_mask"><material>Gazebo/White</material></gazebo>
-    <link name="nose">
+    <link name="left_eye">
         <visual>
             <geometry><sphere radius="0.015"/></geometry>
-            <material name="dora_red"/>
-        </visual>
-    </link>
-    <joint name="nose_joint" type="fixed">
-        <parent link="head"/>
-        <child link="nose"/>
-        <origin xyz="${head_size/2 + 0.01} 0 0.01" rpy="0 0 0"/>
-    </joint>
-    <gazebo reference="nose"><material>Gazebo/Red</material></gazebo>
-    <link name="left_eye">
-        <visual>
-            <geometry><sphere radius="0.018"/></geometry>
-            <material name="dora_white"/>
+            <material name="white"/>
         </visual>
     </link>
@@ -112,10 +75,10 @@
         <parent link="head"/>
         <child link="left_eye"/>
-        <origin xyz="${head_size/2 + 0.005} 0.035 0.035" rpy="0 0 0"/>
+        <origin xyz="${head_size/2} 0.035 0.02" rpy="0 0 0"/>
     </joint>
     <link name="right_eye">
         <visual>
-            <geometry><sphere radius="0.018"/></geometry>
-            <material name="dora_white"/>
+            <geometry><sphere radius="0.015"/></geometry>
+            <material name="white"/>
         </visual>
     </link>
@@ -123,25 +86,25 @@
         <parent link="head"/>
         <child link="right_eye"/>
-        <origin xyz="${head_size/2 + 0.005} -0.035 0.035" rpy="0 0 0"/>
-    </joint>
-    <gazebo reference="left_eye"><material>Gazebo/White</material></gazebo>
-    <gazebo reference="right_eye"><material>Gazebo/White</material></gazebo>
-    <link name="bell">
-        <visual>
-            <geometry><sphere radius="0.025"/></geometry>
-            <material name="dora_yellow"/>
-        </visual>
-    </link>
-    <joint name="bell_joint" type="fixed">
-        <parent link="base_link"/>
-        <child link="bell"/>
-        <origin xyz="${torso_len/2 - 0.02} 0 ${torso_height/2 - 0.02}" rpy="0 0 0"/>
-    </joint>
-    <gazebo reference="bell"><material>Gazebo/Gold</material></gazebo>
+        <origin xyz="${head_size/2} -0.035 0.02" rpy="0 0 0"/>
+    </joint>
+    <gazebo reference="left_eye"><material>Gazebo/Red</material></gazebo>
+    <gazebo reference="right_eye"><material>Gazebo/Red</material></gazebo>
+    <link name="mouth">
+        <visual>
+            <geometry><box size="0.005 0.06 0.02"/></geometry>
+            <material name="red"/>
+        </visual>
+    </link>
+    <joint name="mouth_joint" type="fixed">
+        <parent link="head"/>
+        <child link="mouth"/>
+        <origin xyz="${head_size/2} 0 -0.04" rpy="0 0 0"/>
+    </joint>
+    <gazebo reference="mouth"><material>Gazebo/White</material></gazebo>
     <xacro:macro name="cat_ear" params="prefix y_pos">
         <link name="${prefix}_ear">
             <visual>
                 <geometry><cylinder radius="0.02" length="0.08"/></geometry>
-                <material name="dora_blue"/>
+                <material name="blue"/>
             </visual>
         </link>
@@ -151,5 +114,5 @@
             <origin xyz="0 ${y_pos} ${head_size/2 + 0.04}" rpy="0 0.2 ${y_pos*2}"/>
         </joint>
-        <gazebo reference="${prefix}_ear"><material>Gazebo/SkyBlue</material></gazebo>
+        <gazebo reference="${prefix}_ear"><material>Gazebo/Blue</material></gazebo>
     </xacro:macro>
     <xacro:cat_ear prefix="left" y_pos="0.05"/>
@@ -157,16 +120,16 @@
     <link name="tail">
         <visual>
-            <origin xyz="0.05 0 0" rpy="0 0 0"/>
-            <geometry><sphere radius="0.03"/></geometry>
-            <material name="dora_red"/>
-        </visual>
-        <xacro:sphere_inertia m="0.1" r="0.03"/>
+            <origin xyz="0.15 0 0" rpy="0 1.57 0"/>
+            <geometry><cylinder radius="0.02" length="0.3"/></geometry>
+            <material name="red"/>
+        </visual>
+        <xacro:cylinder_inertia m="0.2" r="0.02" h="0.3"/>
     </link>
     <joint name="tail_joint" type="fixed">
         <parent link="base_link"/>
         <child link="tail"/>
-        <origin xyz="-${torso_len/2} 0 ${torso_height/2}" rpy="0 0 0"/>
-    </joint>
-    <gazebo reference="tail"><material>Gazebo/Red</material></gazebo>
+        <origin xyz="-${torso_len/2} 0 ${torso_height/2}" rpy="0 -0.5 0"/>
+    </joint>
+    <gazebo reference="tail"><material>Gazebo/red</material></gazebo>
     <xacro:macro name="wheel" params="prefix y_pos">
         <link name="${prefix}_wheel">
@@ -188,5 +151,5 @@
             <axis xyz="0 1 0"/>
         </joint>
-        <gazebo reference="${prefix}_wheel"><material>Gazebo/Grey</material></gazebo>
+        <gazebo reference="${prefix}_wheel"><material>Gazebo/silver</material></gazebo>
     </xacro:macro>
     <xacro:wheel prefix="left" y_pos="0.13"/>
@@ -203,9 +166,9 @@
         <origin xyz="0.25 0 -0.05" rpy="0 0 0"/>
     </joint>
-    <gazebo reference="caster_leg"><material>Gazebo/Grey</material></gazebo>
+    <gazebo reference="caster_leg"><material>Gazebo/silver</material></gazebo>
     <link name="front_caster">
         <visual>
             <geometry><sphere radius="${caster_radius}"/></geometry>
-            <material name="white"/>
+            <material name="blue"/>
         </visual>
         <collision>
@@ -219,5 +182,8 @@
         <origin xyz="0 0 -0.04" rpy="0 0 0"/>
     </joint>
-    <gazebo reference="front_caster"><material>Gazebo/White</material></gazebo>
+    <gazebo reference="front_caster">
+        <mu1>0.001</mu1> <mu2>0.001</mu2>
+        <material>Gazebo/Blue</material>
+    </gazebo>
     <link name="lidar_stand">
         <visual>
@@ -257,5 +223,5 @@
             <visualize>true</visualize>
             <update_rate>40</update_rate>
-            <topic>cat/scan</topic>
+            <topic>scan</topic>
             <ray>
                 <scan>
@@ -287,5 +253,5 @@
         <parent link="head"/>
         <child link="camera_link"/>
-        <origin xyz="${head_size/2 + 0.005} 0 0.06" rpy="0 0 0"/>
+        <origin xyz="${head_size/2} 0 0" rpy="0 0 0"/>
     </joint>
     <gazebo reference="camera_link">
@@ -305,5 +271,5 @@
             <update_rate>30</update_rate>
             <visualize>true</visualize>
-            <topic>cat/camera/image_raw</topic>
+            <topic>camera/image_raw</topic>
         </sensor>
     </gazebo>
@@ -321,5 +287,5 @@
             <always_on>true</always_on>
             <update_rate>100</update_rate>
-            <topic>cat/imu</topic>
+            <topic>imu</topic>
         </sensor>
     </gazebo>
@@ -333,8 +299,7 @@
             <wheel_radius>${wheel_radius}</wheel_radius>
             <odom_publish_frequency>50</odom_publish_frequency>
-            <topic>cat/cmd_vel</topic>
-            <odom_topic>cat/odom</odom_topic>
-            <frame_id>cat/odom</frame_id>
-            <child_frame_id>base_link</child_frame_id>
+            <topic>cmd_vel</topic>
+            <odom_topic>odom</odom_topic>
+            <frame_id>odom</frame_id>
         </plugin>
     </gazebo>

File: pac_mouse_pkg/urdf/cat.urdf.xacro (robot description, xacro)
@@ -1,4 +1,4 @@
 <?xml version="1.0"?>
-<robot name="felix_cat" xmlns:xacro="http://www.ros.org/wiki/xacro">
+<robot name="doraemon_cat" xmlns:xacro="http://www.ros.org/wiki/xacro">
     <xacro:property name="torso_len" value="0.4"/>
     <xacro:property name="torso_width" value="0.2"/>
@@ -10,8 +10,9 @@
     <xacro:property name="wheel_mass" value="1.0"/>
     <xacro:property name="caster_radius" value="0.04"/>
-    <material name="blue"> <color rgba="0.16 0.33 0.48 1"/></material>
-    <material name="white"><color rgba="1 1 1 1"/></material>
+    <material name="dora_blue"><color rgba="0.0 0.6 0.9 1"/></material>
+    <material name="dora_white"><color rgba="1 1 1 1"/></material>
+    <material name="dora_red"><color rgba="0.9 0.1 0.1 1"/></material>
+    <material name="dora_yellow"><color rgba="1 0.8 0.1 1"/></material>
     <material name="black"><color rgba="0 0 0 1"/></material>
-    <material name="red"><color rgba="0.6941 0.2471 0.3294 1"/></material>
     <material name="silver"><color rgba="0.75 0.75 0.75 1"/></material>
     <xacro:macro name="box_inertia" params="m x y z">
@@ -42,5 +43,5 @@
         <visual>
             <geometry><box size="${torso_len} ${torso_width} ${torso_height}"/></geometry>
-            <material name="blue"/>
+            <material name="dora_blue"/>
         </visual>
         <collision>
@@ -49,9 +50,21 @@
         <xacro:box_inertia m="${torso_mass}" x="${torso_len}" y="${torso_width}" z="${torso_height}"/>
     </link>
-    <gazebo reference="base_link"><material>Gazebo/Blue</material></gazebo>
+    <gazebo reference="base_link"><material>Gazebo/SkyBlue</material></gazebo>
+    <link name="pocket">
+        <visual>
+            <geometry><box size="0.01 0.14 0.10"/></geometry>
+            <material name="dora_white"/>
+        </visual>
+    </link>
+    <joint name="pocket_joint" type="fixed">
+        <parent link="base_link"/>
+        <child link="pocket"/>
+        <origin xyz="${torso_len/2 + 0.001} 0 0" rpy="0 0 0"/>
+    </joint>
+    <gazebo reference="pocket"><material>Gazebo/White</material></gazebo>
     <link name="head">
         <visual>
             <geometry><box size="${head_size} ${head_size} ${head_size}"/></geometry>
-            <material name="blue"/>
+            <material name="dora_blue"/>
         </visual>
         <collision>
@@ -60,5 +73,5 @@
         <xacro:box_inertia m="1.0" x="${head_size}" y="${head_size}" z="${head_size}"/>
     </link>
-    <gazebo reference="head"><material>Gazebo/Blue</material></gazebo>
+    <gazebo reference="head"><material>Gazebo/SkyBlue</material></gazebo>
     <joint name="neck_joint" type="fixed">
         <parent link="base_link"/>
@@ -66,8 +79,32 @@
         <origin xyz="${torso_len/2 + head_size/2 - 0.05} 0 ${torso_height/2 - head_size/4}" rpy="0 0 0"/>
     </joint>
+    <link name="face_mask">
+        <visual>
+            <geometry><box size="0.01 0.13 0.11"/></geometry>
+            <material name="dora_white"/>
+        </visual>
+    </link>
+    <joint name="face_mask_joint" type="fixed">
+        <parent link="head"/>
+        <child link="face_mask"/>
+        <origin xyz="${head_size/2 + 0.001} 0 -0.01" rpy="0 0 0"/>
+    </joint>
+    <gazebo reference="face_mask"><material>Gazebo/White</material></gazebo>
+    <link name="nose">
+        <visual>
+            <geometry><sphere radius="0.015"/></geometry>
+            <material name="dora_red"/>
+        </visual>
+    </link>
+    <joint name="nose_joint" type="fixed">
+        <parent link="head"/>
+        <child link="nose"/>
+        <origin xyz="${head_size/2 + 0.01} 0 0.01" rpy="0 0 0"/>
+    </joint>
+    <gazebo reference="nose"><material>Gazebo/Red</material></gazebo>
     <link name="left_eye">
         <visual>
-            <geometry><sphere radius="0.015"/></geometry>
-            <material name="white"/>
+            <geometry><sphere radius="0.018"/></geometry>
+            <material name="dora_white"/>
         </visual>
     </link>
@@ -75,10 +112,10 @@
         <parent link="head"/>
         <child link="left_eye"/>
-        <origin xyz="${head_size/2} 0.035 0.02" rpy="0 0 0"/>
+        <origin xyz="${head_size/2 + 0.005} 0.035 0.035" rpy="0 0 0"/>
     </joint>
     <link name="right_eye">
         <visual>
-            <geometry><sphere radius="0.015"/></geometry>
-            <material name="white"/>
+            <geometry><sphere radius="0.018"/></geometry>
+            <material name="dora_white"/>
         </visual>
     </link>
@@ -86,25 +123,25 @@
         <parent link="head"/>
         <child link="right_eye"/>
-        <origin xyz="${head_size/2} -0.035 0.02" rpy="0 0 0"/>
-    </joint>
-    <gazebo reference="left_eye"><material>Gazebo/Red</material></gazebo>
-    <gazebo reference="right_eye"><material>Gazebo/Red</material></gazebo>
-    <link name="mouth">
-        <visual>
-            <geometry><box size="0.005 0.06 0.02"/></geometry>
-            <material name="red"/>
-        </visual>
-    </link>
-    <joint name="mouth_joint" type="fixed">
-        <parent link="head"/>
-        <child link="mouth"/>
-        <origin xyz="${head_size/2} 0 -0.04" rpy="0 0 0"/>
-    </joint>
-    <gazebo reference="mouth"><material>Gazebo/White</material></gazebo>
+        <origin xyz="${head_size/2 + 0.005} -0.035 0.035" rpy="0 0 0"/>
+    </joint>
+    <gazebo reference="left_eye"><material>Gazebo/White</material></gazebo>
+    <gazebo reference="right_eye"><material>Gazebo/White</material></gazebo>
+    <link name="bell">
+        <visual>
+            <geometry><sphere radius="0.025"/></geometry>
+            <material name="dora_yellow"/>
+        </visual>
+    </link>
+    <joint name="bell_joint" type="fixed">
+        <parent link="base_link"/>
+        <child link="bell"/>
+        <origin xyz="${torso_len/2 - 0.02} 0 ${torso_height/2 - 0.02}" rpy="0 0 0"/>
+    </joint>
+    <gazebo reference="bell"><material>Gazebo/Gold</material></gazebo>
     <xacro:macro name="cat_ear" params="prefix y_pos">
         <link name="${prefix}_ear">
             <visual>
                 <geometry><cylinder radius="0.02" length="0.08"/></geometry>
-                <material name="blue"/>
+                <material name="dora_blue"/>
             </visual>
         </link>
@@ -114,5 +151,5 @@
             <origin xyz="0 ${y_pos} ${head_size/2 + 0.04}" rpy="0 0.2 ${y_pos*2}"/>
         </joint>
-        <gazebo reference="${prefix}_ear"><material>Gazebo/Blue</material></gazebo>
+        <gazebo reference="${prefix}_ear"><material>Gazebo/SkyBlue</material></gazebo>
     </xacro:macro>
     <xacro:cat_ear prefix="left" y_pos="0.05"/>
@@ -120,16 +157,16 @@
     <link name="tail">
         <visual>
-            <origin xyz="0.15 0 0" rpy="0 1.57 0"/>
-            <geometry><cylinder radius="0.02" length="0.3"/></geometry>
-            <material name="red"/>
-        </visual>
-        <xacro:cylinder_inertia m="0.2" r="0.02" h="0.3"/>
+            <origin xyz="0.05 0 0" rpy="0 0 0"/>
+            <geometry><sphere radius="0.03"/></geometry>
+            <material name="dora_red"/>
+        </visual>
+        <xacro:sphere_inertia m="0.1" r="0.03"/>
     </link>
     <joint name="tail_joint" type="fixed">
         <parent link="base_link"/>
         <child link="tail"/>
-        <origin xyz="-${torso_len/2} 0 ${torso_height/2}" rpy="0 -0.5 0"/>
-    </joint>
-    <gazebo reference="tail"><material>Gazebo/red</material></gazebo>
+        <origin xyz="-${torso_len/2} 0 ${torso_height/2}" rpy="0 0 0"/>
+    </joint>
+    <gazebo reference="tail"><material>Gazebo/Red</material></gazebo>
     <xacro:macro name="wheel" params="prefix y_pos">
         <link name="${prefix}_wheel">
@@ -151,5 +188,5 @@
             <axis xyz="0 1 0"/>
         </joint>
-        <gazebo reference="${prefix}_wheel"><material>Gazebo/silver</material></gazebo>
+        <gazebo reference="${prefix}_wheel"><material>Gazebo/Grey</material></gazebo>
     </xacro:macro>
     <xacro:wheel prefix="left" y_pos="0.13"/>
@@ -166,9 +203,9 @@
         <origin xyz="0.25 0 -0.05" rpy="0 0 0"/>
     </joint>
-    <gazebo reference="caster_leg"><material>Gazebo/silver</material></gazebo>
+    <gazebo reference="caster_leg"><material>Gazebo/Grey</material></gazebo>
     <link name="front_caster">
         <visual>
             <geometry><sphere radius="${caster_radius}"/></geometry>
-            <material name="blue"/>
+            <material name="white"/>
         </visual>
         <collision>
@@ -182,8 +219,5 @@
         <origin xyz="0 0 -0.04" rpy="0 0 0"/>
     </joint>
-    <gazebo reference="front_caster">
-        <mu1>0.001</mu1> <mu2>0.001</mu2>
-        <material>Gazebo/Blue</material>
-    </gazebo>
+    <gazebo reference="front_caster"><material>Gazebo/White</material></gazebo>
     <link name="lidar_stand">
         <visual>
@@ -223,5 +257,5 @@
             <visualize>true</visualize>
             <update_rate>40</update_rate>
-            <topic>scan</topic>
+            <topic>cat/scan</topic>
             <ray>
                 <scan>
@@ -253,5 +287,5 @@
         <parent link="head"/>
         <child link="camera_link"/>
-        <origin xyz="${head_size/2} 0 0" rpy="0 0 0"/>
+        <origin xyz="${head_size/2 + 0.005} 0 0.06" rpy="0 0 0"/>
     </joint>
     <gazebo reference="camera_link">
@@ -271,5 +305,5 @@
             <update_rate>30</update_rate>
             <visualize>true</visualize>
-            <topic>camera/image_raw</topic>
+            <topic>cat/camera/image_raw</topic>
         </sensor>
     </gazebo>
@@ -287,5 +321,5 @@
             <always_on>true</always_on>
             <update_rate>100</update_rate>
-            <topic>imu</topic>
+            <topic>cat/imu</topic>
         </sensor>
     </gazebo>
@@ -299,7 +333,8 @@
             <wheel_radius>${wheel_radius}</wheel_radius>
             <odom_publish_frequency>50</odom_publish_frequency>
-            <topic>cmd_vel</topic>
-            <odom_topic>odom</odom_topic>
-            <frame_id>odom</frame_id>
+            <topic>cat/cmd_vel</topic>
+            <odom_topic>cat/odom</odom_topic>
+            <frame_id>cat/odom</frame_id>
+            <child_frame_id>base_link</child_frame_id>
         </plugin>
     </gazebo>
