Commit message: Update cat robot URDF and simulation launch config
Refactored cat.urdf.xacro to remove caster wheels, adjust base and sensor positions, and update Gazebo plugin parameters for improved simulation stability. Updated final_simulation.launch.py to use cat_fixed.urdf.xacro, set safe spawn positions, fix camera topic bridges, and add frame_prefix for state publishers. Simplified RViz config to focus on LiDAR and camera topics, and set fixed frame to mouse_robot/odom.

File: pac_mouse_pkg/urdf/cat.urdf.xacro (robot description, xacro)
@@ -4,5 +4,5 @@
   <xacro:property name="base_width" value="0.25"/>
   <xacro:property name="base_length" value="0.30"/>
-  <xacro:property name="base_height" value="0.12"/>
+  <xacro:property name="base_height" value="0.10"/>
   <xacro:property name="base_mass" value="2.0"/>
   <xacro:property name="wheel_radius" value="0.05"/>
@@ -10,7 +10,5 @@
   <xacro:property name="wheel_mass" value="0.3"/>
   <xacro:property name="wheel_separation" value="0.25"/>
-  <xacro:property name="caster_radius" value="0.025"/>
-  <xacro:property name="caster_mass" value="0.1"/>
-  <!-- MATERIALS (Red and White for Cat) -->
+  <!-- MATERIALS -->
   <material name="red">
     <color rgba="0.8 0.0 0.0 1.0"/>
@@ -25,5 +23,5 @@
   <link name="base_link">
     <visual>
-      <origin xyz="0 0 0" rpy="0 0 0"/>
+      <origin xyz="0 0 0.05" rpy="0 0 0"/>
       <geometry>
         <box size="${base_length} ${base_width} ${base_height}"/>
@@ -32,5 +30,5 @@
     </visual>
     <collision>
-      <origin xyz="0 0 0" rpy="0 0 0"/>
+      <origin xyz="0 0 0.05" rpy="0 0 0"/>
       <geometry>
         <box size="${base_length} ${base_width} ${base_height}"/>
@@ -38,9 +36,8 @@
     </collision>
     <inertial>
-      <origin xyz="0 0 0" rpy="0 0 0"/>
+      <origin xyz="0 0 0.05" rpy="0 0 0"/>
       <mass value="${base_mass}"/>
       <inertia ixx="${(1/12) * base_mass * (base_width*base_width + base_height*base_height)}"
-               ixy="0.0"
-               ixz="0.0"
+               ixy="0.0" ixz="0.0"
                iyy="${(1/12) * base_mass * (base_length*base_length + base_height*base_height)}"
                iyz="0.0"
@@ -48,5 +45,5 @@
     </inertial>
   </link>
-  <!-- CAT EARS (Visual Only - Makes it look like a cat) -->
+  <!-- CAT EARS -->
   <link name="left_ear">
     <visual>
@@ -65,5 +62,5 @@
     <parent link="base_link"/>
     <child link="left_ear"/>
-    <origin xyz="0.10 0.08 ${base_height/2 + 0.03}" rpy="0 0.3 0"/>
+    <origin xyz="0.10 0.08 ${base_height + 0.03}" rpy="0 0.3 0"/>
   </joint>
   <link name="right_ear">
@@ -83,5 +80,5 @@
     <parent link="base_link"/>
     <child link="right_ear"/>
-    <origin xyz="0.10 -0.08 ${base_height/2 + 0.03}" rpy="0 0.3 0"/>
+    <origin xyz="0.10 -0.08 ${base_height + 0.03}" rpy="0 0.3 0"/>
   </joint>
   <!-- LEFT WHEEL -->
@@ -104,6 +101,5 @@
       <mass value="${wheel_mass}"/>
       <inertia ixx="${(1/12) * wheel_mass * (3*wheel_radius*wheel_radius + wheel_width*wheel_width)}"
-               ixy="0.0"
-               ixz="0.0"
+               ixy="0.0" ixz="0.0"
                iyy="${(1/12) * wheel_mass * (3*wheel_radius*wheel_radius + wheel_width*wheel_width)}"
                iyz="0.0"
@@ -114,5 +110,5 @@
     <parent link="base_link"/>
     <child link="left_wheel"/>
-    <origin xyz="0 ${wheel_separation/2} ${-base_height/2 + wheel_radius}" rpy="0 0 0"/>
+    <origin xyz="0 ${wheel_separation/2} 0" rpy="0 0 0"/>
     <axis xyz="0 1 0"/>
   </joint>
@@ -136,6 +132,5 @@
       <mass value="${wheel_mass}"/>
       <inertia ixx="${(1/12) * wheel_mass * (3*wheel_radius*wheel_radius + wheel_width*wheel_width)}"
-               ixy="0.0"
-               ixz="0.0"
+               ixy="0.0" ixz="0.0"
                iyy="${(1/12) * wheel_mass * (3*wheel_radius*wheel_radius + wheel_width*wheel_width)}"
                iyz="0.0"
@@ -146,84 +141,6 @@
     <parent link="base_link"/>
     <child link="right_wheel"/>
-    <origin xyz="0 ${-wheel_separation/2} ${-base_height/2 + wheel_radius}" rpy="0 0 0"/>
+    <origin xyz="0 ${-wheel_separation/2} 0" rpy="0 0 0"/>
     <axis xyz="0 1 0"/>
-  </joint>
-  <!-- FRONT CASTER -->
-  <link name="front_caster">
-    <visual>
-      <origin xyz="0 0 0" rpy="0 0 0"/>
-      <geometry>
-        <sphere radius="${caster_radius}"/>
-      </geometry>
-      <material name="white"/>
-    </visual>
-    <collision>
-      <origin xyz="0 0 0" rpy="0 0 0"/>
-      <geometry>
-        <sphere radius="${caster_radius}"/>
-      </geometry>
-      <surface>
-        <friction>
-          <ode>
-            <mu>0.01</mu>
-            <mu2>0.01</mu2>
-          </ode>
-        </friction>
-      </surface>
-    </collision>
-    <inertial>
-      <origin xyz="0 0 0" rpy="0 0 0"/>
-      <mass value="${caster_mass}"/>
-      <inertia ixx="${(2/5) * caster_mass * caster_radius * caster_radius}"
-               ixy="0.0"
-               ixz="0.0"
-               iyy="${(2/5) * caster_mass * caster_radius * caster_radius}"
-               iyz="0.0"
-               izz="${(2/5) * caster_mass * caster_radius * caster_radius}"/>
-    </inertial>
-  </link>
-  <joint name="front_caster_joint" type="fixed">
-    <parent link="base_link"/>
-    <child link="front_caster"/>
-    <origin xyz="${base_length/3} 0 ${-base_height/2 - caster_radius + 0.01}" rpy="0 0 0"/>
-  </joint>
-  <!-- REAR CASTER -->
-  <link name="rear_caster">
-    <visual>
-      <origin xyz="0 0 0" rpy="0 0 0"/>
-      <geometry>
-        <sphere radius="${caster_radius}"/>
-      </geometry>
-      <material name="white"/>
-    </visual>
-    <collision>
-      <origin xyz="0 0 0" rpy="0 0 0"/>
-      <geometry>
-        <sphere radius="${caster_radius}"/>
-      </geometry>
-      <surface>
-        <friction>
-          <ode>
-            <mu>0.01</mu>
-            <mu2>0.01</mu2>
-          </ode>
-        </friction>
-      </surface>
-    </collision>
-    <inertial>
-      <origin xyz="0 0 0" rpy="0 0 0"/>
-      <mass value="${caster_mass}"/>
-      <inertia ixx="${(2/5) * caster_mass * caster_radius * caster_radius}"
-               ixy="0.0"
-               ixz="0.0"
-               iyy="${(2/5) * caster_mass * caster_radius * caster_radius}"
-               iyz="0.0"
-               izz="${(2/5) * caster_mass * caster_radius * caster_radius}"/>
-    </inertial>
-  </link>
-  <joint name="rear_caster_joint" type="fixed">
-    <parent link="base_link"/>
-    <child link="rear_caster"/>
-    <origin xyz="${-base_length/3} 0 ${-base_height/2 - caster_radius + 0.01}" rpy="0 0 0"/>
   </joint>
   <!-- LIDAR LINK -->
@@ -236,10 +153,4 @@
       <material name="black"/>
     </visual>
-    <collision>
-      <origin xyz="0 0 0" rpy="0 0 0"/>
-      <geometry>
-        <cylinder radius="0.04" length="0.05"/>
-      </geometry>
-    </collision>
     <inertial>
       <mass value="0.15"/>
@@ -250,5 +161,5 @@
     <parent link="base_link"/>
     <child link="lidar_link"/>
-    <origin xyz="0.05 0 ${base_height/2 + 0.05}" rpy="0 0 0"/>
+    <origin xyz="0.05 0 ${base_height + 0.05}" rpy="0 0 0"/>
   </joint>
   <!-- CAMERA LINK -->
@@ -261,10 +172,4 @@
       <material name="black"/>
     </visual>
-    <collision>
-      <origin xyz="0 0 0" rpy="0 0 0"/>
-      <geometry>
-        <box size="0.03 0.08 0.03"/>
-      </geometry>
-    </collision>
     <inertial>
       <mass value="0.1"/>
@@ -275,5 +180,5 @@
     <parent link="base_link"/>
     <child link="camera_link"/>
-    <origin xyz="${base_length/2} 0 0.02" rpy="0 0 0"/>
+    <origin xyz="${base_length/2} 0 0.05" rpy="0 0 0"/>
   </joint>
   <!-- IMU LINK -->
@@ -289,12 +194,9 @@
     <origin xyz="0 0 0" rpy="0 0 0"/>
   </joint>
-  <!-- ========================================= -->
-  <!-- GAZEBO PLUGINS -->
-  <!-- ========================================= -->
-  <!-- Gazebo colors -->
+  <!-- GAZEBO PROPERTIES -->
   <gazebo reference="base_link">
     <material>Gazebo/Red</material>
-    <mu1>0.3</mu1>
-    <mu2>0.3</mu2>
+    <mu1>0.1</mu1>
+    <mu2>0.1</mu2>
   </gazebo>
   <gazebo reference="left_ear">
@@ -308,4 +210,6 @@
     <mu1>1.0</mu1>
     <mu2>1.0</mu2>
+    <kp>1000000.0</kp>
+    <kd>100.0</kd>
   </gazebo>
   <gazebo reference="right_wheel">
@@ -313,19 +217,11 @@
     <mu1>1.0</mu1>
     <mu2>1.0</mu2>
-  </gazebo>
-  <gazebo reference="front_caster">
-    <material>Gazebo/White</material>
-    <mu1>0.001</mu1>
-    <mu2>0.001</mu2>
-  </gazebo>
-  <gazebo reference="rear_caster">
-    <material>Gazebo/White</material>
-    <mu1>0.001</mu1>
-    <mu2>0.001</mu2>
+    <kp>1000000.0</kp>
+    <kd>100.0</kd>
   </gazebo>
   <gazebo reference="lidar_link">
     <material>Gazebo/Black</material>
   </gazebo>
-  <!-- LIDAR SENSOR PLUGIN -->
+  <!-- LIDAR SENSOR -->
   <gazebo reference="lidar_link">
     <sensor name="cat_lidar" type="gpu_lidar">
@@ -333,5 +229,4 @@
       <topic>cat/scan</topic>
       <update_rate>10</update_rate>
-      <enable_metrics>false</enable_metrics>
       <lidar>
         <scan>
@@ -346,11 +241,5 @@
           <min>0.15</min>
           <max>12.0</max>
-          <resolution>0.01</resolution>
         </range>
-        <noise>
-          <type>gaussian</type>
-          <mean>0.0</mean>
-          <stddev>0.01</stddev>
-        </noise>
       </lidar>
       <always_on>true</always_on>
@@ -358,9 +247,9 @@
     </sensor>
   </gazebo>
-  <!-- CAMERA SENSOR PLUGIN -->
+  <!-- CAMERA SENSOR -->
   <gazebo reference="camera_link">
     <sensor name="cat_camera" type="camera">
       <pose>0 0 0 0 0 0</pose>
-      <topic>cat/camera/image_raw</topic>
+      <topic>cat/camera</topic>
       <update_rate>30</update_rate>
       <camera>
@@ -375,15 +264,10 @@
           <far>100</far>
         </clip>
-        <noise>
-          <type>gaussian</type>
-          <mean>0.0</mean>
-          <stddev>0.007</stddev>
-        </noise>
       </camera>
       <always_on>true</always_on>
-      <visualize>true</visualize>
+      <visualize>false</visualize>
     </sensor>
   </gazebo>
-  <!-- IMU SENSOR PLUGIN -->
+  <!-- IMU SENSOR -->
   <gazebo reference="imu_link">
     <sensor name="cat_imu" type="imu">
@@ -391,49 +275,7 @@
       <update_rate>100</update_rate>
       <always_on>true</always_on>
-      <imu>
-        <angular_velocity>
-          <x>
-            <noise type="gaussian">
-              <mean>0.0</mean>
-              <stddev>0.01</stddev>
-            </noise>
-          </x>
-          <y>
-            <noise type="gaussian">
-              <mean>0.0</mean>
-              <stddev>0.01</stddev>
-            </noise>
-          </y>
-          <z>
-            <noise type="gaussian">
-              <mean>0.0</mean>
-              <stddev>0.01</stddev>
-            </noise>
-          </z>
-        </angular_velocity>
-        <linear_acceleration>
-          <x>
-            <noise type="gaussian">
-              <mean>0.0</mean>
-              <stddev>0.1</stddev>
-            </noise>
-          </x>
-          <y>
-            <noise type="gaussian">
-              <mean>0.0</mean>
-              <stddev>0.1</stddev>
-            </noise>
-          </y>
-          <z>
-            <noise type="gaussian">
-              <mean>0.0</mean>
-              <stddev>0.1</stddev>
-            </noise>
-          </z>
-        </linear_acceleration>
-      </imu>
     </sensor>
   </gazebo>
-  <!-- DIFFERENTIAL DRIVE PLUGIN -->
+  <!-- DIFFERENTIAL DRIVE -->
   <gazebo>
     <plugin filename="gz-sim-diff-drive-system" name="gz::sim::systems::DiffDrive">
@@ -448,5 +290,5 @@
       <odom_topic>cat/odom</odom_topic>
       <frame_id>odom</frame_id>
-      <child_frame_id>base_link</child_frame_id>
+      <child_frame_id>cat_robot/base_link</child_frame_id>
     </plugin>
   </gazebo>

Commit message: Add origin to inertial macros and caster inertia
Added <origin> tags to the box_inertia, cylinder_inertia, and sphere_inertia macros to explicitly define the inertial frame. Also added missing inertia to the caster_wheel link for improved physical accuracy.

File: pac_mouse_pkg/urdf/cat.urdf.xacro (robot description, xacro)
@@ -18,5 +18,5 @@
     <xacro:macro name="box_inertia" params="m x y z">
         <inertial>
-            <mass value="${m}"/>
+            <origin xyz="0 0 0" rpy="0 0 0"/> <mass value="${m}"/>
             <inertia ixx="${m*(y*y+z*z)/12}" ixy="0" ixz="0"
                      iyy="${m*(x*x+z*z)/12}" iyz="0"
@@ -26,5 +26,5 @@
     <xacro:macro name="cylinder_inertia" params="m r h">
         <inertial>
-            <mass value="${m}"/>
+            <origin xyz="0 0 0" rpy="0 0 0"/> <mass value="${m}"/>
             <inertia ixx="${m*(3*r*r+h*h)/12}" ixy="0" ixz="0"
                      iyy="${m*(3*r*r+h*h)/12}" iyz="0"
@@ -34,5 +34,5 @@
     <xacro:macro name="sphere_inertia" params="m r">
         <inertial>
-            <mass value="${m}"/>
+            <origin xyz="0 0 0" rpy="0 0 0"/> <mass value="${m}"/>
             <inertia ixx="${2*m*r*r/5}" ixy="0" ixz="0"
                      iyy="${2*m*r*r/5}" iyz="0"
@@ -197,4 +197,5 @@
             <material name="silver"/>
         </visual>
+        <xacro:cylinder_inertia m="0.1" r="0.02" h="0.05"/>
     </link>
     <joint name="caster_leg_joint" type="fixed">

Commit message: Replace xacro inertia macro with explicit inertial tag
Replaces the use of <xacro:cylinder_inertia> with an explicit <inertial> tag for the relevant link in cat.urdf.xacro. This change provides direct control over the inertia parameters and improves URDF clarity.

File: pac_mouse_pkg/urdf/cat.urdf.xacro (robot description, xacro)
@@ -197,5 +197,8 @@
             <material name="silver"/>
         </visual>
-        <xacro:cylinder_inertia m="0.1" r="0.02" h="0.05"/>
+        <inertial>
+            <origin xyz="0 0 0" rpy="0 0 0"/>
+            <mass value="0.1"/> <inertia ixx="0.0001" ixy="0" ixz="0" iyy="0.0001" iyz="0" izz="0.0001"/>
+        </inertial>
     </link>
     <joint name="caster_leg_joint" type="fixed">
