Commit message: Trying to lower COG of Mouse

File: pac_mouse_pkg/urdf/mouse.urdf.xacro (robot description, xacro)
@@ -5,5 +5,5 @@
     <xacro:property name="body_width" value="0.10"/>
     <xacro:property name="body_height" value="0.06"/>
-    <xacro:property name="body_mass" value="0.5"/>
+    <xacro:property name="body_mass" value="2"/>
     <xacro:property name="wheel_radius" value="0.035"/>
     <xacro:property name="wheel_width" value="0.01"/>
@@ -14,8 +14,8 @@
     <xacro:macro name="box_inertia" params="m x y z">
         <inertial>
-            <mass value="${m}"/>
-            <inertia ixx="${m*(y*y+z*z)/12}" ixy="0" ixz="0"
-                     iyy="${m*(x*x+z*z)/12}" iyz="0"
-                     izz="${m*(x*x+y*y)/12}"/>
+        <mass value="${m}"/>
+            <origin xyz="0 0 ${o_z}" rpy="0 0 0"/> <inertia ixx="${m*(y*y+z*z)/12}" ixy="0" ixz="0"
+                    iyy="${m*(x*x+z*z)/12}" iyz="0"
+                    izz="${m*(x*x+y*y)/12}"/>
         </inertial>
     </xacro:macro>
@@ -44,5 +44,5 @@
             <geometry><box size="${body_len} ${body_width} ${body_height}"/></geometry>
         </collision>
-        <xacro:box_inertia m="${body_mass}" x="${body_len}" y="${body_width}" z="${body_height}"/>
+        <xacro:box_inertia m="${body_mass}" x="${body_len}" y="${body_width}" z="${body_height}" o_z="-0.05"/>
     </link>
     <gazebo reference="$(arg robot_name)/base_link">
@@ -237,5 +237,5 @@
             <topic>/model/$(arg robot_name)/odometry</topic>
             <tf_topic>/model/$(arg robot_name)/tf</tf_topic>
-            <odom_frame>map</odom_frame>
+            <odom_frame>$(arg robot_name)/odom</odom_frame>
             <robot_base_frame>$(arg robot_name)/base_link</robot_base_frame>
             <odom_publish_frequency>50</odom_publish_frequency>

Commit message: Update mouse.urdf.xacro

File: pac_mouse_pkg/urdf/mouse.urdf.xacro (robot description, xacro)
@@ -14,8 +14,8 @@
     <xacro:macro name="box_inertia" params="m x y z">
         <inertial>
-        <mass value="${m}"/>
-            <origin xyz="0 0 ${o_z}" rpy="0 0 0"/> <inertia ixx="${m*(y*y+z*z)/12}" ixy="0" ixz="0"
-                    iyy="${m*(x*x+z*z)/12}" iyz="0"
-                    izz="${m*(x*x+y*y)/12}"/>
+            <mass value="${m}"/>
+            <inertia ixx="${m*(y*y+z*z)/12}" ixy="0" ixz="0"
+                     iyy="${m*(x*x+z*z)/12}" iyz="0"
+                     izz="${m*(x*x+y*y)/12}"/>
         </inertial>
     </xacro:macro>
@@ -44,5 +44,5 @@
             <geometry><box size="${body_len} ${body_width} ${body_height}"/></geometry>
         </collision>
-        <xacro:box_inertia m="${body_mass}" x="${body_len}" y="${body_width}" z="${body_height}" o_z="-0.05"/>
+        <xacro:box_inertia m="${body_mass}" x="${body_len}" y="${body_width}" z="${body_height}"/>
     </link>
     <gazebo reference="$(arg robot_name)/base_link">

Commit message: Update mouse.urdf.xacro

File: pac_mouse_pkg/urdf/mouse.urdf.xacro (robot description, xacro)
@@ -44,5 +44,12 @@
             <geometry><box size="${body_len} ${body_width} ${body_height}"/></geometry>
         </collision>
-        <xacro:box_inertia m="${body_mass}" x="${body_len}" y="${body_width}" z="${body_height}"/>
+        <inertial>
+            <mass value="2.0"/>
+            <origin xyz="0 0 -0.05" rpy="0 0 0"/>
+            <inertia
+                ixx="${2.0*(body_width*body_width + body_height*body_height)/12}" ixy="0" ixz="0"
+                iyy="${2.0*(body_len*body_len + body_height*body_height)/12}" iyz="0"
+                izz="${2.0*(body_len*body_len + body_width*body_width)/12}"/>
+        </inertial>
     </link>
     <gazebo reference="$(arg robot_name)/base_link">

Commit message: Update mouse.urdf.xacro

File: pac_mouse_pkg/urdf/mouse.urdf.xacro (robot description, xacro)
@@ -145,5 +145,5 @@
         <parent link="$(arg robot_name)/base_link"/>
         <child link="$(arg robot_name)/lidar_link"/>
-        <origin xyz="0 0 ${body_height/2 + 0.01}" rpy="0 0 0"/>
+        <origin xyz="0 0 ${body_height/2 + 0.01}" rpy="0 0.04 0"/>
     </joint>
     <gazebo reference="$(arg robot_name)/lidar_link">

Commit message: Update mouse.urdf.xacro

File: pac_mouse_pkg/urdf/mouse.urdf.xacro (robot description, xacro)
@@ -145,5 +145,5 @@
         <parent link="$(arg robot_name)/base_link"/>
         <child link="$(arg robot_name)/lidar_link"/>
-        <origin xyz="0 0 ${body_height/2 + 0.01}" rpy="0 0.04 0"/>
+        <origin xyz="0 0 ${body_height/2 + 0.01}" rpy="0 0.03 0"/>
     </joint>
     <gazebo reference="$(arg robot_name)/lidar_link">

Commit message: testing wheel effort.

File: pac_mouse_pkg/urdf/mouse.urdf.xacro (robot description, xacro)
@@ -105,4 +105,5 @@
             <child link="$(arg robot_name)/${prefix}_wheel"/>
             <origin xyz="0.03 ${y_pos} -0.02" rpy="0 0 0"/> <axis xyz="0 1 0"/>
+            <limit effort="100" velocity="20.0"/>
         </joint>
         <gazebo reference="$(arg robot_name)/${prefix}_wheel">
